File: hardware/car.kicad_sch (KiCad schematic)
At the start: 25 parts, among them M1 motor FL, M2 motor RL, M3 motor RR, M4 motor FR, SW1 E-stop (NC, optional), U1 ESP32-S3-CAM (N16R8) - Freeno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, U2 Raspberry Pi Pico (RP2040) - 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, U3 SparkFun ROB-14450 #1 (left: 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, U4 SparkFun ROB-14450 #2 (right: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, U5 BMI160 breakout, U6 PCM5102A DAC (on-board 3V3 re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, U7 PAM8302A class-D amp

Commit message: Carro con audio
Parts:
- removed D1: BAT54 Schottky, symbol car:D-Schottky
- added R7: 0R link (no Schottky), symbol car:R
- R3, R4: value 4.7k I2C pull-up (DNP?) -> 4.7k pull-up (DO NOT FIT)
- U5: value BMI160 breakout -> BMI160 breakout (VIN 3-5 V; own 3V3 reg + 3.9k pull-ups)
Connections:
- net +3V3_S3: no longer U5.1 (VDD), U5.2 (VDDIO), U5.4 (CS)
- net +5V: now also U5.VIN, R7.1
- net DRV2_AIN1: now also U2.15 (GP11); no longer U2.10 (GP7)
- net DRV2_AIN2: now also U2.16 (GP12); no longer U2.11 (GP8)
- net DRV2_BIN1: now also U2.19 (GP14); no longer U2.14 (GP10)
- net DRV2_BIN2: now also U2.17 (GP13); no longer U2.12 (GP9)
- net DRV2_PWMA: now also U2.14 (GP10); no longer U2.9 (GP6)
- net DRV2_PWMB: now also U2.20 (GP15); no longer U2.15 (GP11)
- net GND: now also U5.GND; no longer U5.3 (GND), U5.7 (SDO)
- net I2C_SCL: now also U1.R5 (GPIO42 MTMS), U5.SCL; no longer U1.R4 (GPIO2 ADC1_CH1), U5.6 (SCL)
- net I2C_SDA: now also U1.R6 (GPIO41 MTDI), U5.SDA; no longer U1.R3 (GPIO1 ADC1_CH0), U5.5 (SDA)
- net I2S_BCK: now also U1.R16 (GPIO47); no longer U1.R15 (GPIO48 WS2812)
- net I2S_DIN: now also U1.R17 (GPIO21); no longer U1.R16 (GPIO47)
- net I2S_LRCK: now also U1.R14 (GPIO45 VSPI); no longer U1.R17 (GPIO21)
- net S3_LED: now also U1.R15 (GPIO48 WS2812); no longer U1.R14 (GPIO45 VSPI)
- net VSYS: now also R7.2
- no-connect marks 53 -> 60

Commit message: controllers communication
Connections:
- net LINK_RX_S3: now also U1.R4 (GPIO2 ADC1_CH1); no longer U1.R2 (GPIO44 U0RXD)
- net S3_TXD: now also U1.R3 (GPIO1 ADC1_CH0); no longer U1.R1 (GPIO43 U0TXD)
Changed lines of the file:
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@@
     (instances
       (project "car"
-        (path "/b6ef7c33-35d0-442f-82e3-3e8c832db472" (reference "U1") (unit 1))
+        (path "/07895b60-07f5-48f8-97ed-c2c0ef5051ec" (reference "U1") (unit 1))
       )
     )
@@
     (effects (font (size 1.27 1.27)) (justify right bottom))
   )
-  (wire (pts (xy 87.63 44.45) (xy 92.71 44.45))
-    (stroke (width 0) (type default))
-  )
-  (label "S3_TXD" (at 92.71 44.45 0)
-    (effects (font (size 1.27 1.27)) (justify left bottom))
-  )
-  (wire (pts (xy 87.63 46.99) (xy 92.71 46.99))
-    (stroke (width 0) (type default))
-  )
-  (label "LINK_RX_S3" (at 92.71 46.99 0)
-    (effects (font (size 1.27 1.27)) (justify left bottom))
-  )
-  (no_connect (at 87.63 49.53))
-  (no_connect (at 87.63 52.07))
+  (no_connect (at 87.63 44.45))
+  (no_connect (at 87.63 46.99))
+  (wire (pts (xy 87.63 49.53) (xy 92.71 49.53))
+    (stroke (width 0) (type default))
+  )
+  (label "S3_TXD" (at 92.71 49.53 0)
+    (effects (font (size 1.27 1.27)) (justify left bottom))
+  )
+  (wire (pts (xy 87.63 52.07) (xy 92.71 52.07))
+    (stroke (width 0) (type default))
+  )
+  (label "LINK_RX_S3" (at 92.71 52.07 0)
+    (effects (font (size 1.27 1.27)) (justify left bottom))
+  )
   (wire (pts (xy 87.63 54.61) (xy 92.71 54.61))
     (stroke (width 0) (type default))
@@
     (instances
       (project "car"
-        (path "/b6ef7c33-35d0-442f-82e3-3e8c832db472" (reference "U2") (unit 1))
+        (path "/07895b60-07f5-48f8-97ed-c2c0ef5051ec" (reference "U2") (unit 1))
       )
     )
@@
     (instances
       (project "car"
-        (path "/b6ef7c33-35d0-442f-82e3-3e8c832db472" (reference "U3") (unit 1))
+        (path "/07895b60-07f5-48f8-97ed-c2c0ef5051ec" (reference "U3") (unit 1))
       )
     )
@@
     (instances
       (project "car"
-        (path "/b6ef7c33-35d0-442f-82e3-3e8c832db472" (reference "U4") (unit 1))
+        (path "/07895b60-07f5-48f8-97ed-c2c0ef5051ec" (reference "U4") (unit 1))
       )
     )
@@
     (instances
       (project "car"
-        (path "/b6ef7c33-35d0-442f-82e3-3e8c832db472" (reference "U5") (unit 1))
+        (path "/07895b60-07f5-48f8-97ed-c2c0ef5051ec" (reference "U5") (unit 1))
       )
     )
@@
     (instances
       (project "car"
-        (path "/b6ef7c33-35d0-442f-82e3-3e8c832db472" (reference "U6") (unit 1))
+        (path "/07895b60-07f5-48f8-97ed-c2c0ef5051ec" (reference "U6") (unit 1))
       )
     )
@@
     (instances
       (project "car"
-        (path "/b6ef7c33-35d0-442f-82e3-3e8c832db472" (reference "U7") (unit 1))
+        (path "/07895b60-07f5-48f8-97ed-c2c0ef5051ec" (reference "U7") (unit 1))
       )
     )
@@
     (instances
       (project "car"
-        (path "/b6ef7c33-35d0-442f-82e3-3e8c832db472" (reference "PS1") (unit 1))
+        (path "/07895b60-07f5-48f8-97ed-c2c0ef5051ec" (reference "PS1") (unit 1))
       )
     )
@@
     (instances
       (project "car"
-        (path "/b6ef7c33-35d0-442f-82e3-3e8c832db472" (reference "PS2") (unit 1))
+        (path "/07895b60-07f5-48f8-97ed-c2c0ef5051ec" (reference "PS2") (unit 1))
       )
     )
@@
     (instances
       (project "car"
-        (path "/b6ef7c33-35d0-442f-82e3-3e8c832db472" (reference "BT1") (unit 1))
+        (path "/07895b60-07f5-48f8-97ed-c2c0ef5051ec" (reference "BT1") (unit 1))
       )
     )
@@
     (instances
       (project "car"
-        (path "/b6ef7c33-35d0-442f-82e3-3e8c832db472" (reference "F1") (unit 1))
+        (path "/07895b60-07f5-48f8-97ed-c2c0ef5051ec" (reference "F1") (unit 1))
       )
     )
@@
     (instances
       (project "car"
-        (path "/b6ef7c33-35d0-442f-82e3-3e8c832db472" (reference "R7") (unit 1))
+        (path "/07895b60-07f5-48f8-97ed-c2c0ef5051ec" (reference "R7") (unit 1))
       )
     )
@@
     (instances
       (project "car"
-        (path "/b6ef7c33-35d0-442f-82e3-3e8c832db472" (reference "R1") (unit 1))
+        (path "/07895b60-07f5-48f8-97ed-c2c0ef5051ec" (reference "R1") (unit 1))
       )
     )
@@
     (instances
       (project "car"
-        (path "/b6ef7c33-35d0-442f-82e3-3e8c832db472" (reference "R2") (unit 1))
+        (path "/07895b60-07f5-48f8-97ed-c2c0ef5051ec" (reference "R2") (unit 1))
       )
     )
@@
     (instances
       (project "car"
-        (path "/b6ef7c33-35d0-442f-82e3-3e8c832db472" (reference "R3") (unit 1))
+        (path "/07895b60-07f5-48f8-97ed-c2c0ef5051ec" (reference "R3") (unit 1))
       )
     )
@@
     (instances
       (project "car"
-        (path "/b6ef7c33-35d0-442f-82e3-3e8c832db472" (reference "R4") (unit 1))
+        (path "/07895b60-07f5-48f8-97ed-c2c0ef5051ec" (reference "R4") (unit 1))
       )
     )
@@
     (instances
       (project "car"
-        (path "/b6ef7c33-35d0-442f-82e3-3e8c832db472" (reference "R5") (unit 1))
+        (path "/07895b60-07f5-48f8-97ed-c2c0ef5051ec" (reference "R5") (unit 1))
       )
     )
@@
     (instances
       (project "car"
-        (path "/b6ef7c33-35d0-442f-82e3-3e8c832db472" (reference "R6") (unit 1))
+        (path "/07895b60-07f5-48f8-97ed-c2c0ef5051ec" (reference "R6") (unit 1))
       )
     )
@@
     (instances
       (project "car"
-        (path "/b6ef7c33-35d0-442f-82e3-3e8c832db472" (reference "SW1") (unit 1))
+        (path "/07895b60-07f5-48f8-97ed-c2c0ef5051ec" (reference "SW1") (unit 1))
       )
     )
@@
     (instances
       (project "car"
-        (path "/b6ef7c33-35d0-442f-82e3-3e8c832db472" (reference "M1") (unit 1))
+        (path "/07895b60-07f5-48f8-97ed-c2c0ef5051ec" (reference "M1") (unit 1))
       )
     )
@@
     (instances
       (project "car"
-        (path "/b6ef7c33-35d0-442f-82e3-3e8c832db472" (reference "M2") (unit 1))
+        (path "/07895b60-07f5-48f8-97ed-c2c0ef5051ec" (reference "M2") (unit 1))
       )
     )
@@
     (instances
       (project "car"
-        (path "/b6ef7c33-35d0-442f-82e3-3e8c832db472" (reference "M3") (unit 1))
+        (path "/07895b60-07f5-48f8-97ed-c2c0ef5051ec" (reference "M3") (unit 1))
       )
     )
@@
     (instances
       (project "car"
-        (path "/b6ef7c33-35d0-442f-82e3-3e8c832db472" (reference "M4") (unit 1))
+        (path "/07895b60-07f5-48f8-97ed-c2c0ef5051ec" (reference "M4") (unit 1))
       )
     )
@@
     (instances
       (project "car"
-        (path "/b6ef7c33-35d0-442f-82e3-3e8c832db472" (reference "LED1") (unit 1))
+        (path "/07895b60-07f5-48f8-97ed-c2c0ef5051ec" (reference "LED1") (unit 1))
       )
     )
@@
     (instances
       (project "car"
-        (path "/b6ef7c33-35d0-442f-82e3-3e8c832db472" (reference "SP1") (unit 1))
-      )
-    )
+        (path "/07895b60-07f5-48f8-97ed-c2c0ef5051ec" (reference "SP1") (unit 1))
+      )
+    )
